File: hardware/eeprom_emu_16bit.kicad_sch (KiCad schematic)
At the start: 4 parts, among them U3 74HCT02, U4 74HCT00

Commit message: Hardware: Drew up the rest of the pcb
Parts:
- added H1, H2, H3, H4: MountingHole, MountingHole:MountingHole_3.2mm_M3_ISO7380_Pad, symbol Mechanical:MountingHole
- gave numbers to parts that had none: 2
