File: hardware/extconn.kicad_sch (KiCad schematic)
At the start: 21 parts, among them J3 Conn_02x20_Odd_Even, U3 74HCT02, U4 74HCT00, U5 74HCT541, U6 74HCT541, U7 74HCT541, U8 74HCT541, U9 74HCT541

Commit message: Hardware: Drew up the rest of the pcb
Parts:
- added R4, R5, R6: 10k, Resistor_SMD:R_0805_2012Metric_Pad1.20x1.40mm_HandSolder, symbol Device:R_Small
- C4, C5: value C_Small -> 0.1uF; footprint (none) -> Capacitor_SMD:C_1206_3216Metric_Pad1.33x1.80mm_HandSolder
- gave numbers to parts that had none: 8
Connections:
- net EVENSEL: now also R6.1
- net GND: now also J3.34 (Pin_34), R4.1, R5.2, R6.2
- net ODDSEL: now also R5.1
- net OE: now also R4.2
- net D0: now reaches U5.2 (A0)
- net D1: now reaches U5.3 (A1)
- net D2: now reaches U5.4 (A2)
- net D3: now reaches U5.5 (A3)
- net D4: now reaches U5.6 (A4)
- net D5: now reaches U5.7 (A5)
- net D6: now reaches U5.8 (A6)
- net D7: now reaches U5.9 (A7)
- net D8: now reaches U6.2 (A0)
- net D9: now reaches U6.3 (A1)
- net D10: now reaches U6.4 (A2)
- net D11: now reaches U6.5 (A3)
- net D12: now reaches U6.6 (A4)
- net D13: now reaches U6.7 (A5)
- net D14: now reaches U6.8 (A6)
- net D15: now reaches U6.9 (A7)
- no-connect marks 6 -> 5
