File: hardware/mcu.kicad_sch (KiCad schematic)
At the start: 18 parts, among them J1 USB_OTG, J2 Conn_01x03_Male, U1 CH340C, U2 ATmega3209-A

Commit message: Hardware: Drew up the rest of the pcb
Parts:
- J2: footprint (none) -> Connector_PinHeader_2.54mm:PinHeader_1x03_P2.54mm_Vertical
- gave numbers to parts that had none: 10
Changed lines of the file:
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@@
   (symbol (lib_id "power:+5V") (at 64.77 25.4 270) (unit 1)
     (in_bom yes) (on_board yes) (fields_autoplaced)
-    (property "Reference" "#PWR?" (id 0) (at 60.96 25.4 0)
+    (property "Reference" "#PWR0120" (id 0) (at 60.96 25.4 0)
       (effects (font (size 1.27 1.27)) hide)
     )
@@
   (symbol (lib_id "Device:C_Small") (at 104.14 97.155 90) (unit 1)
     (in_bom yes) (on_board yes) (fields_autoplaced)
-    (property "Reference" "C?" (id 0) (at 104.1463 91.8931 90))
+    (property "Reference" "C12" (id 0) (at 104.1463 91.8931 90))
     (property "Value" "0.1uF" (id 1) (at 104.1463 94.43 90))
     (property "Footprint" "Capacitor_SMD:C_1206_3216Metric_Pad1.33x1.80mm_HandSolder" (id 2) (at 104.14 97.155 0)
@@
   (symbol (lib_id "power:GND") (at 97.79 142.24 0) (unit 1)
     (in_bom yes) (on_board yes) (fields_autoplaced)
-    (property "Reference" "#PWR?" (id 0) (at 97.79 148.59 0)
+    (property "Reference" "#PWR0114" (id 0) (at 97.79 148.59 0)
       (effects (font (size 1.27 1.27)) hide)
     )
@@
   (symbol (lib_id "power:+5V") (at 60.325 55.245 0) (unit 1)
     (in_bom yes) (on_board yes) (fields_autoplaced)
-    (property "Reference" "#PWR?" (id 0) (at 60.325 59.055 0)
+    (property "Reference" "#PWR0118" (id 0) (at 60.325 59.055 0)
       (effects (font (size 1.27 1.27)) hide)
     )
@@
   (symbol (lib_id "Device:LED") (at 36.83 25.4 0) (unit 1)
     (in_bom yes) (on_board yes)
-    (property "Reference" "D?" (id 0) (at 37.465 29.21 0))
+    (property "Reference" "D1" (id 0) (at 37.465 29.21 0))
     (property "Value" "LED GREEN" (id 1) (at 37.465 31.115 0))
     (property "Footprint" "LED_SMD:LED_0805_2012Metric_Pad1.15x1.40mm_HandSolder" (id 2) (at 36.83 25.4 0)
@@
   (symbol (lib_id "power:GND") (at 60.325 98.425 90) (unit 1)
     (in_bom yes) (on_board yes) (fields_autoplaced)
-    (property "Reference" "#PWR?" (id 0) (at 66.675 98.425 0)
+    (property "Reference" "#PWR0122" (id 0) (at 66.675 98.425 0)
       (effects (font (size 1.27 1.27)) hide)
     )
@@
   (symbol (lib_id "Device:R_Small") (at 53.975 25.4 90) (unit 1)
     (in_bom yes) (on_board yes)
-    (property "Reference" "R?" (id 0) (at 53.975 23.495 90))
+    (property "Reference" "R2" (id 0) (at 53.975 23.495 90))
     (property "Value" "470" (id 1) (at 53.975 21.59 90))
     (property "Footprint" "Resistor_SMD:R_0805_2012Metric_Pad1.20x1.40mm_HandSolder" (id 2) (at 53.975 25.4 0)
@@
   (symbol (lib_id "power:+5V") (at 76.2 78.105 0) (unit 1)
     (in_bom yes) (on_board yes) (fields_autoplaced)
-    (property "Reference" "#PWR?" (id 0) (at 76.2 81.915 0)
+    (property "Reference" "#PWR0116" (id 0) (at 76.2 81.915 0)
       (effects (font (size 1.27 1.27)) hide)
     )
@@
   (symbol (lib_id "power:GND") (at 48.26 143.51 0) (unit 1)
     (in_bom yes) (on_board yes) (fields_autoplaced)
-    (property "Reference" "#PWR?" (id 0) (at 48.26 149.86 0)
+    (property "Reference" "#PWR0115" (id 0) (at 48.26 149.86 0)
       (effects (font (size 1.27 1.27)) hide)
     )
@@
   (symbol (lib_id "74xx:74HCT541") (at 97.79 120.65 0) (mirror y) (unit 1)
     (in_bom yes) (on_board yes) (fields_autoplaced)
-    (property "Reference" "U?" (id 0) (at 98.3106 101.7102 0)
+    (property "Reference" "U11" (id 0) (at 98.3106 101.7102 0)
       (effects (font (size 1.27 1.27)) (justify right))
     )
@@
   (symbol (lib_id "Switch:SW_MEC_5E") (at 88.9 81.915 0) (unit 1)
     (in_bom yes) (on_board yes) (fields_autoplaced)
-    (property "Reference" "SW?" (id 0) (at 88.9 72.7542 0))
+    (property "Reference" "SW1" (id 0) (at 88.9 72.7542 0))
     (property "Value" "SW_MEC_5E" (id 1) (at 88.9 75.2911 0))
     (property "Footprint" "Button_Switch_THT:SW_PUSH_6mm_H4.3mm" (id 2) (at 88.9 74.295 0)
@@
   (symbol (lib_id "power:GND") (at 60.325 70.485 0) (unit 1)
     (in_bom yes) (on_board yes) (fields_autoplaced)
-    (property "Reference" "#PWR?" (id 0) (at 60.325 76.835 0)
+    (property "Reference" "#PWR0117" (id 0) (at 60.325 76.835 0)
       (effects (font (size 1.27 1.27)) hide)
     )
@@
   (symbol (lib_id "power:+5V") (at 48.26 95.25 0) (unit 1)
     (in_bom yes) (on_board yes) (fields_autoplaced)
-    (property "Reference" "#PWR?" (id 0) (at 48.26 99.06 0)
+    (property "Reference" "#PWR0121" (id 0) (at 48.26 99.06 0)
       (effects (font (size 1.27 1.27)) hide)
     )
@@
   (symbol (lib_id "power:GND") (at 114.3 76.2 270) (unit 1)
     (in_bom yes) (on_board yes) (fields_autoplaced)
-    (property "Reference" "#PWR?" (id 0) (at 107.95 76.2 0)
+    (property "Reference" "#PWR0111" (id 0) (at 107.95 76.2 0)
       (effects (font (size 1.27 1.27)) hide)
     )
@@
   (symbol (lib_id "Power_Protection:SP0505BAHT") (at 60.325 62.865 0) (unit 1)
     (in_bom yes) (on_board yes) (fields_autoplaced)
-    (property "Reference" "D?" (id 0) (at 68.072 62.0303 0)
+    (property "Reference" "D2" (id 0) (at 68.072 62.0303 0)
       (effects (font (size 1.27 1.27)) (justify left))
     )
@@
   (symbol (lib_id "Device:R_Small") (at 129.54 76.2 90) (unit 1)
     (in_bom yes) (on_board yes)
-    (property "Reference" "R?" (id 0) (at 129.54 80.645 90))
+    (property "Reference" "R3" (id 0) (at 129.54 80.645 90))
     (property "Value" "470" (id 1) (at 129.54 78.74 90))
     (property "Footprint" "Resistor_SMD:R_0805_2012Metric_Pad1.20x1.40mm_HandSolder" (id 2) (at 129.54 76.2 0)
@@
   (symbol (lib_id "Device:C_Small") (at 55.245 98.425 90) (unit 1)
     (in_bom yes) (on_board yes) (fields_autoplaced)
-    (property "Reference" "C?" (id 0) (at 55.2513 93.1631 90))
+    (property "Reference" "C11" (id 0) (at 55.2513 93.1631 90))
     (property "Value" "0.1uF" (id 1) (at 55.2513 95.7 90))
     (property "Footprint" "Capacitor_SMD:C_1206_3216Metric_Pad1.33x1.80mm_HandSolder" (id 2) (at 55.245 98.425 0)
@@
   (symbol (lib_id "Device:LED") (at 120.65 76.2 0) (unit 1)
     (in_bom yes) (on_board yes)
-    (property "Reference" "D?" (id 0) (at 121.285 78.74 0))
+    (property "Reference" "D3" (id 0) (at 121.285 78.74 0))
     (property "Value" "LED RED" (id 1) (at 120.65 80.645 0))
     (property "Footprint" "LED_SMD:LED_0805_2012Metric_Pad1.15x1.40mm_HandSolder" (id 2) (at 120.65 76.2 0)
@@
     (property "Reference" "J2" (id 0) (at 129.54 38.261 90))
     (property "Value" "Conn_01x03_Male" (id 1) (at 129.54 40.7979 90))
-    (property "Footprint" "" (id 2) (at 129.54 41.91 0)
+    (property "Footprint" "Connector_PinHeader_2.54mm:PinHeader_1x03_P2.54mm_Vertical" (id 2) (at 129.54 41.91 0)
       (effects (font (size 1.27 1.27)) hide)
     )
@@
   (symbol (lib_id "power:GND") (at 31.115 25.4 270) (unit 1)
     (in_bom yes) (on_board yes) (fields_autoplaced)
-    (property "Reference" "#PWR?" (id 0) (at 24.765 25.4 0)
+    (property "Reference" "#PWR0119" (id 0) (at 24.765 25.4 0)
       (effects (font (size 1.27 1.27)) hide)
     )
@@
   (symbol (lib_id "74xx:74HCT541") (at 48.26 121.92 0) (mirror y) (unit 1)
     (in_bom yes) (on_board yes) (fields_autoplaced)
-    (property "Reference" "U?" (id 0) (at 48.7806 102.9802 0)
+    (property "Reference" "U10" (id 0) (at 48.7806 102.9802 0)
       (effects (font (size 1.27 1.27)) (justify right))
     )
@@
   (symbol (lib_id "power:+5V") (at 97.79 95.25 0) (unit 1)
     (in_bom yes) (on_board yes) (fields_autoplaced)
-    (property "Reference" "#PWR?" (id 0) (at 97.79 99.06 0)
+    (property "Reference" "#PWR0113" (id 0) (at 97.79 99.06 0)
       (effects (font (size 1.27 1.27)) hide)
     )
@@
   (symbol (lib_id "power:GND") (at 109.855 97.155 90) (unit 1)
     (in_bom yes) (on_board yes) (fields_autoplaced)
-    (property "Reference" "#PWR?" (id 0) (at 116.205 97.155 0)
-      (effects (font (size 1.27 1.27)) hide)
-    )
+    (property "Reference" "#PWR0112" (id 0) (at 116.205 97.155 0)
+      (effects (font (size 1.27 1.27)) hide)
+    )
