File: hardware/memory.kicad_sch (KiCad schematic)
At the start: 4 parts

Commit message: Hardware: Drew up the rest of the pcb
Parts:
- gave numbers to parts that had none: 4
Changed lines of the file:
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@@
   (symbol (lib_id "power:GND") (at 187.325 60.96 90) (unit 1)
     (in_bom yes) (on_board yes) (fields_autoplaced)
-    (property "Reference" "#PWR?" (id 0) (at 193.675 60.96 0)
+    (property "Reference" "#PWR0132" (id 0) (at 193.675 60.96 0)
       (effects (font (size 1.27 1.27)) hide)
     )
@@
   (symbol (lib_id "power:+5V") (at 98.425 56.515 0) (unit 1)
     (in_bom yes) (on_board yes) (fields_autoplaced)
-    (property "Reference" "#PWR?" (id 0) (at 98.425 60.325 0)
+    (property "Reference" "#PWR0134" (id 0) (at 98.425 60.325 0)
       (effects (font (size 1.27 1.27)) hide)
     )
@@
   (symbol (lib_id "power:GND") (at 175.895 127 0) (unit 1)
     (in_bom yes) (on_board yes) (fields_autoplaced)
-    (property "Reference" "#PWR?" (id 0) (at 175.895 133.35 0)
+    (property "Reference" "#PWR0131" (id 0) (at 175.895 133.35 0)
       (effects (font (size 1.27 1.27)) hide)
     )
@@
   (symbol (lib_id "Memory_RAM:AS6C4008-55PCN") (at 98.425 94.615 0) (unit 1)
     (in_bom yes) (on_board yes) (fields_autoplaced)
-    (property "Reference" "U?" (id 0) (at 100.4444 65.5152 0)
+    (property "Reference" "U12" (id 0) (at 100.4444 65.5152 0)
       (effects (font (size 1.27 1.27)) (justify left))
     )
@@
   (symbol (lib_id "power:GND") (at 98.425 126.365 0) (unit 1)
     (in_bom yes) (on_board yes) (fields_autoplaced)
-    (property "Reference" "#PWR?" (id 0) (at 98.425 132.715 0)
+    (property "Reference" "#PWR0136" (id 0) (at 98.425 132.715 0)
       (effects (font (size 1.27 1.27)) hide)
     )
@@
   (symbol (lib_id "power:+5V") (at 175.895 57.15 0) (unit 1)
     (in_bom yes) (on_board yes) (fields_autoplaced)
-    (property "Reference" "#PWR?" (id 0) (at 175.895 60.96 0)
+    (property "Reference" "#PWR0133" (id 0) (at 175.895 60.96 0)
       (effects (font (size 1.27 1.27)) hide)
     )
@@
   (symbol (lib_id "Device:C_Small") (at 105.41 59.69 90) (unit 1)
     (in_bom yes) (on_board yes) (fields_autoplaced)
-    (property "Reference" "C?" (id 0) (at 105.4163 54.4281 90))
+    (property "Reference" "C13" (id 0) (at 105.4163 54.4281 90))
     (property "Value" "0.1uF" (id 1) (at 105.4163 56.965 90))
     (property "Footprint" "Capacitor_SMD:C_1206_3216Metric_Pad1.33x1.80mm_HandSolder" (id 2) (at 105.41 59.69 0)
@@
   (symbol (lib_id "Memory_RAM:AS6C4008-55PCN") (at 175.895 95.885 0) (unit 1)
     (in_bom yes) (on_board yes) (fields_autoplaced)
-    (property "Reference" "U?" (id 0) (at 177.9144 66.7852 0)
+    (property "Reference" "U13" (id 0) (at 177.9144 66.7852 0)
       (effects (font (size 1.27 1.27)) (justify left))
     )
@@
   (symbol (lib_id "power:GND") (at 111.76 59.69 90) (unit 1)
     (in_bom yes) (on_board yes) (fields_autoplaced)
-    (property "Reference" "#PWR?" (id 0) (at 118.11 59.69 0)
+    (property "Reference" "#PWR0135" (id 0) (at 118.11 59.69 0)
       (effects (font (size 1.27 1.27)) hide)
     )
@@
   (symbol (lib_id "Device:C_Small") (at 181.61 60.96 90) (unit 1)
     (in_bom yes) (on_board yes) (fields_autoplaced)
-    (property "Reference" "C?" (id 0) (at 181.6163 55.6981 90))
+    (property "Reference" "C14" (id 0) (at 181.6163 55.6981 90))
     (property "Value" "0.1uF" (id 1) (at 181.6163 58.235 90))
     (property "Footprint" "Capacitor_SMD:C_1206_3216Metric_Pad1.33x1.80mm_HandSolder" (id 2) (at 181.61 60.96 0)
